Commit message: changes in urdf

File: urdf/gazebo_control.xacro (robot description, xacro)
@@ -5,7 +5,6 @@
             <ros>
                 <namespace>rav_bot</namespace>
-                <argument>cmd_vel</argument>
             </ros>
-            <robotNamespace>rav_bot</robotNamespace>
+            <updateRate>10</updateRate>
             <!-- Wheel Information -->
             <left_joint>left_wheel_joint</left_joint>
@@ -14,12 +13,15 @@
             <wheel_diameter>0.066</wheel_diameter>
             <!-- Limits -->
-            <max_wheel_torque>200</max_wheel_torque>
-            <max_wheel_acceleration>10.0</max_wheel_acceleration>
+            <max_wheel_torque>20</max_wheel_torque>
+            <max_wheel_acceleration>1.0</max_wheel_acceleration>
+            <commandTopic>cmd_vel</commandTopic>
             <!-- Output -->
-            <odometry_frame>odom</odometry_frame>
-            <robot_base_frame>base_link</robot_base_frame>
-            <publish_odom>true</publish_odom>
-            <publish_odom_tf>true</publish_odom_tf>
-            <publish_wheel_tf>true</publish_wheel_tf>
+            <publishOdom>true</publishOdom>
+            <publishOdomTf>false</publishOdomTf>
+            <publisherWheelTf>true</publisherWheelTf>
+            <odomFrame>odom</odomFrame>
+            <odom_base_frame>base_link</odom_base_frame>
+            <!-- set true for swap wheels -->
+            <!-- <legacyMode>false</legacyMode>  -->
         </plugin>
     </gazebo>

File: urdf/robot.urdf.xacro (robot description, xacro)
@@ -5,4 +5,5 @@
     <xacro:include filename="robot_core.xacro" />
     <xacro:include filename="gazebo_control.xacro"/>
+    <xacro:include filename="inertial_macros.xacro"/>
     <!-- <xacro:if value="$(arg use_ros2_control)">
         <xacro:include filename="ros2_control.xacro" />
@@ -13,4 +14,5 @@
     <xacro:include filename="lidar.xacro" />
     <xacro:include filename="camera.xacro" />
+    <xacro:include filename="imu.xacro"/>
     <!-- <xacro:include filename="depth_camera.xacro" /> -->
 </robot>

File: urdf/robot_core.xacro (robot description, xacro)
@@ -38,6 +38,6 @@
     <!-- BASE_FOOTPRINT LINK -->
     <joint name="base_footprint_joint" type="fixed">
-        <parent link="base_footprint"/>
-        <child link="base_link"/>
+        <parent link="base_link"/>
+        <child link="base_footprint"/>
         <origin xyz="0 0 0.033" rpy="0 0 0"/>
     </joint>
